File: blocks/power/usb_c_5v/usb_c_5v.kicad_sch (KiCad schematic)
At the start: 3 parts, among them J1 USB-C 16P

Commit message: R12 최종: 표기를 자유 텍스트로 전환 — 왼쪽 정렬 고정 (사용자 지적)
'심볼 왼쪽 끝에 정렬, 삐져나오면 안 이쁘다' — 회전 심볼의 속성 텍스트는
커널이 정렬·위치를 재계산해 좌표 예측이 불가함을 실측으로 확인. 명시
배치 모드에서는 속성(Reference/Value)을 숨기고 자유 텍스트 요소로 그린다:
- 짝의 왼쪽 끝 일치 (justify left, 같은 x), 행간 2.03
- J1/U1은 심볼 왼쪽 모서리에 정렬, 수동소자는 부품 옆 좌측 정렬 열
전 게이트 PASS (블록 3개)
Other:
- note added: "5.1kΩ"
- note added: "J1"
- note added: "R1"
- note added: "R2"
- note added: "USB-C 16P"
Changed lines of the file:
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@@
 		(color 0 0 0 0)
+	)
+	(text "J1"
+		(exclude_from_sim no)
+		(at 53.34 49.02 0)
+		(effects
+			(font
+				(size 1.27 1.27)
+			)
+			(justify left)
+		)
+	)
+	(text "USB-C 16P"
+		(exclude_from_sim no)
+		(at 53.34 51.05 0)
+		(effects
+			(font
+				(size 1.27 1.27)
+			)
+			(justify left)
+		)
+	)
+	(text "R1"
+		(exclude_from_sim no)
+		(at 27.94 70.49 0)
+		(effects
+			(font
+				(size 1.27 1.27)
+			)
+			(justify left)
+		)
+	)
+	(text "5.1kΩ"
+		(exclude_from_sim no)
+		(at 27.94 72.52 0)
+		(effects
+			(font
+				(size 1.27 1.27)
+			)
+			(justify left)
+		)
+	)
+	(text "R2"
+		(exclude_from_sim no)
+		(at 88.67 70.49 0)
+		(effects
+			(font
+				(size 1.27 1.27)
+			)
+			(justify left)
+		)
+	)
+	(text "5.1kΩ"
+		(exclude_from_sim no)
+		(at 88.67 72.52 0)
+		(effects
+			(font
+				(size 1.27 1.27)
+			)
+			(justify left)
+		)
 	)
 	(hierarchical_label "USB_DP"
@@
 		(dnp no)
 		(property "Reference" "J1"
-			(at 63.5 49.02 0)
-			(effects
-				(font
-					(size 1.27 1.27)
-				)
+			(at 53.34 49.02 0)
+			(effects
+				(font
+					(size 1.27 1.27)
+				)
+				(hide yes)
 			)
 		)
 		(property "Value" "USB-C 16P"
-			(at 63.5 51.05 0)
-			(effects
-				(font
-					(size 1.27 1.27)
-				)
+			(at 53.34 51.05 0)
+			(effects
+				(font
+					(size 1.27 1.27)
+				)
+				(hide yes)
 			)
 		)
@@
 		(dnp no)
 		(property "Reference" "R1"
-			(at 26.67 70.49 0)
-			(effects
-				(font
-					(size 1.27 1.27)
-				)
+			(at 27.94 70.49 0)
+			(effects
+				(font
+					(size 1.27 1.27)
+				)
+				(hide yes)
 			)
 		)
 		(property "Value" "5.1kΩ"
-			(at 26.67 72.52 0)
-			(effects
-				(font
-					(size 1.27 1.27)
-				)
+			(at 27.94 72.52 0)
+			(effects
+				(font
+					(size 1.27 1.27)
+				)
+				(hide yes)
 			)
 		)
@@
 		(dnp no)
 		(property "Reference" "R2"
-			(at 90.8 70.49 0)
-			(effects
-				(font
-					(size 1.27 1.27)
-				)
+			(at 88.67 70.49 0)
+			(effects
+				(font
+					(size 1.27 1.27)
+				)
+				(hide yes)
 			)
 		)
 		(property "Value" "5.1kΩ"
-			(at 90.8 72.52 0)
-			(effects
-				(font
-					(size 1.27 1.27)
-				)
-			)
-		)
+			(at 88.67 72.52 0)
+			(effects
+				(font
+					(size 1.27 1.27)
+				)
+				(hide yes)
+			)
+		)
