File: dist/design_blocks/PartReel.kicad_blocks/cortex_debug_10.kicad_block/cortex_debug_10.kicad_sch (KiCad schematic)
At the start: 1 part, among them J1 Cortex Debug 10P

Commit message: 디자인 블록 재배포: g431_min 0.2(VBAT 100nF C8), emi_power_in·buck_24v_5v P13 limit_mm 실측 보정 (boardworks g431_ind24 T2)
Co-Authored-By: Claude Fable 5 <noreply@anthropic.com>
Other:
- title: Cortex debug connector (10-pin 1.27mm) -> cortex_debug_10
Changed lines of the file:
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@@
 	(paper "A5")
 	(title_block
-		(title "Cortex debug connector (10-pin 1.27mm)")
+		(title "cortex_debug_10")
 		(company "PartReel block")
 		(rev "0.1")
@@
 			)
 		)
-		(column_widths 12.4 42.4)
+		(column_widths 13.3 48.1)
 		(row_heights 4.45 4.45 4.45 4.45 4.45 4.45 4.45 4.45 4.45 4.45 4.45)
 		(cells
 			(table_cell "Block"
 				(exclude_from_sim no)
-				(at 133.35 68.58 0)
-				(size 12.4 4.45)
+				(at 134.62 71.12 0)
+				(size 13.3 4.45)
 				(margins 0.9525 0.9525 0.9525 0.9525)
 				(span 1 1)
@@
 			(table_cell "Cortex debug connector (10-pin 1.27mm)"
 				(exclude_from_sim no)
-				(at 145.75 68.58 0)
-				(size 42.4 4.45)
+				(at 147.92 71.12 0)
+				(size 48.1 4.45)
 				(margins 0.9525 0.9525 0.9525 0.9525)
 				(span 1 1)
@@
 			(table_cell "Rev"
 				(exclude_from_sim no)
-				(at 133.35 73.03 0)
-				(size 12.4 4.45)
+				(at 134.62 75.57 0)
+				(size 13.3 4.45)
 				(margins 0.9525 0.9525 0.9525 0.9525)
 				(span 1 1)
@@
 			(table_cell "0.1"
 				(exclude_from_sim no)
-				(at 145.75 73.03 0)
-				(size 42.4 4.45)
+				(at 147.92 75.57 0)
+				(size 48.1 4.45)
 				(margins 0.9525 0.9525 0.9525 0.9525)
 				(span 1 1)
@@
 			(table_cell "PWR In"
 				(exclude_from_sim no)
-				(at 133.35 77.48 0)
-				(size 12.4 4.45)
+				(at 134.62 80.02 0)
+				(size 13.3 4.45)
 				(margins 0.9525 0.9525 0.9525 0.9525)
 				(span 1 1)
@@
 			(table_cell "+3V3, GND"
 				(exclude_from_sim no)
-				(at 145.75 77.48 0)
-				(size 42.4 4.45)
+				(at 147.92 80.02 0)
+				(size 48.1 4.45)
 				(margins 0.9525 0.9525 0.9525 0.9525)
 				(span 1 1)
@@
 			(table_cell "In"
 				(exclude_from_sim no)
-				(at 133.35 81.93 0)
-				(size 12.4 4.45)
+				(at 134.62 84.47 0)
+				(size 13.3 4.45)
 				(margins 0.9525 0.9525 0.9525 0.9525)
 				(span 1 1)
@@
 			(table_cell "SWO"
 				(exclude_from_sim no)
-				(at 145.75 81.93 0)
-				(size 42.4 4.45)
+				(at 147.92 84.47 0)
+				(size 48.1 4.45)
 				(margins 0.9525 0.9525 0.9525 0.9525)
 				(span 1 1)
@@
 			(table_cell "Out"
 				(exclude_from_sim no)
-				(at 133.35 86.38 0)
-				(size 12.4 4.45)
+				(at 134.62 88.92 0)
+				(size 13.3 4.45)
 				(margins 0.9525 0.9525 0.9525 0.9525)
 				(span 1 1)
@@
 			(table_cell "NRST, SWCLK"
 				(exclude_from_sim no)
-				(at 145.75 86.38 0)
-				(size 42.4 4.45)
+				(at 147.92 88.92 0)
+				(size 48.1 4.45)
 				(margins 0.9525 0.9525 0.9525 0.9525)
 				(span 1 1)
@@
 			(table_cell "I/O"
 				(exclude_from_sim no)
-				(at 133.35 90.83 0)
-				(size 12.4 4.45)
+				(at 134.62 93.37 0)
+				(size 13.3 4.45)
 				(margins 0.9525 0.9525 0.9525 0.9525)
 				(span 1 1)
@@
 			(table_cell "SWDIO"
 				(exclude_from_sim no)
-				(at 145.75 90.83 0)
-				(size 42.4 4.45)
+				(at 147.92 93.37 0)
+				(size 48.1 4.45)
 				(margins 0.9525 0.9525 0.9525 0.9525)
 				(span 1 1)
@@
 			(table_cell "Connector"
 				(exclude_from_sim no)
-				(at 133.35 95.28 0)
-				(size 12.4 4.45)
+				(at 134.62 97.82 0)
+				(size 13.3 4.45)
 				(margins 0.9525 0.9525 0.9525 0.9525)
 				(span 1 1)
@@
 			(table_cell "FTSH-105-01-L-DV-007-K"
 				(exclude_from_sim no)
-				(at 145.75 95.28 0)
-				(size 42.4 4.45)
+				(at 147.92 97.82 0)
+				(size 48.1 4.45)
 				(margins 0.9525 0.9525 0.9525 0.9525)
 				(span 1 1)
@@
 			(table_cell "Pitch"
 				(exclude_from_sim no)
-				(at 133.35 99.73 0)
-				(size 12.4 4.45)
+				(at 134.62 102.27 0)
+				(size 13.3 4.45)
 				(margins 0.9525 0.9525 0.9525 0.9525)
 				(span 1 1)
@@
 			(table_cell "1.27mm 2x5"
 				(exclude_from_sim no)
-				(at 145.75 99.73 0)
-				(size 42.4 4.45)
+				(at 147.92 102.27 0)
+				(size 48.1 4.45)
 				(margins 0.9525 0.9525 0.9525 0.9525)
 				(span 1 1)
@@
 			(table_cell "Pin 7"
 				(exclude_from_sim no)
-				(at 133.35 104.18 0)
-				(size 12.4 4.45)
+				(at 134.62 106.72 0)
+				(size 13.3 4.45)
 				(margins 0.9525 0.9525 0.9525 0.9525)
 				(span 1 1)
@@
 			(table_cell "KEY (no pin) - NC"
 				(exclude_from_sim no)
-				(at 145.75 104.18 0)
-				(size 42.4 4.45)
+				(at 147.92 106.72 0)
+				(size 48.1 4.45)
 				(margins 0.9525 0.9525 0.9525 0.9525)
 				(span 1 1)
@@
 			(table_cell "Pin 9"
 				(exclude_from_sim no)
-				(at 133.35 108.63 0)
-				(size 12.4 4.45)
+				(at 134.62 111.17 0)
+				(size 13.3 4.45)
 				(margins 0.9525 0.9525 0.9525 0.9525)
 				(span 1 1)
@@
 			(table_cell "GNDDetect - tied to GND"
 				(exclude_from_sim no)
-				(at 145.75 108.63 0)
-				(size 42.4 4.45)
+				(at 147.92 111.17 0)
+				(size 48.1 4.45)
 				(margins 0.9525 0.9525 0.9525 0.9525)
 				(span 1 1)
@@
 			(table_cell "Source"
 				(exclude_from_sim no)
-				(at 133.35 113.08 0)
-				(size 12.4 4.45)
+				(at 134.62 115.62 0)
+				(size 13.3 4.45)
 				(margins 0.9525 0.9525 0.9525 0.9525)
 				(span 1 1)
@@
 			(table_cell "Arm UG 101636"
 				(exclude_from_sim no)
-				(at 145.75 113.08 0)
-				(size 42.4 4.45)
-				(margins 0.9525 0.9525 0.9525 0.9525)
-				(span 1 1)
+				(at 147.92 115.62 0)
+				(size 48.1 4.45)
+				(margins 0.9525 0.9525 0.9525 0.9525)
+				(span 1 1)
