File: dist/design_blocks/PartReel.kicad_blocks/g431_min.kicad_block/g431_min.kicad_sch (KiCad schematic)
At the start: 9 parts, among them U1 STM32G431CBTx

Commit message: 디자인 블록 재배포: g431_min 0.2(VBAT 100nF C8), emi_power_in·buck_24v_5v P13 limit_mm 실측 보정 (boardworks g431_ind24 T2)
Co-Authored-By: Claude Fable 5 <noreply@anthropic.com>
Parts:
- added C8: 100nF, PCM_PartReel:antmicro_cl05a104ka5nnnc, symbol PartReel:C_100n_25V_0402
Connections:
- net +3V3: now also C8.2
- net GND: now also C8.1
Other:
- note added: "C8"
- title: STM32G431 minimum circuit -> g431_min
