File: dist/design_blocks/PartReel.kicad_blocks/i2c_pullup.kicad_block/i2c_pullup.kicad_sch (KiCad schematic)
At the start: 2 parts

Commit message: 디자인 블록 재배포: g431_min 0.2(VBAT 100nF C8), emi_power_in·buck_24v_5v P13 limit_mm 실측 보정 (boardworks g431_ind24 T2)
Co-Authored-By: Claude Fable 5 <noreply@anthropic.com>
Other:
- title: I2C pull-up (3.3V, 1.8k) -> i2c_pullup
Changed lines of the file:
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@@
 	(paper "A5")
 	(title_block
-		(title "I2C pull-up (3.3V, 1.8k)")
+		(title "i2c_pullup")
 		(company "PartReel block")
-		(rev "0.2")
+		(rev "0.3")
 	)
 	(wire
@@
 			)
 		)
-		(column_widths 10.2 27.7)
+		(column_widths 10.9 31.3)
 		(row_heights 4.45 4.45 4.45 4.45 4.45 4.45 4.45 4.45)
 		(cells
 			(table_cell "Block"
 				(exclude_from_sim no)
-				(at 95.25 45.72 0)
-				(size 10.2 4.45)
+				(at 93.98 45.72 0)
+				(size 10.9 4.45)
 				(margins 0.9525 0.9525 0.9525 0.9525)
 				(span 1 1)
@@
 			(table_cell "I2C pull-up (3.3V, 1.8k)"
 				(exclude_from_sim no)
-				(at 105.45 45.72 0)
-				(size 27.7 4.45)
+				(at 104.88 45.72 0)
+				(size 31.3 4.45)
 				(margins 0.9525 0.9525 0.9525 0.9525)
 				(span 1 1)
@@
 			(table_cell "Rev"
 				(exclude_from_sim no)
-				(at 95.25 50.17 0)
-				(size 10.2 4.45)
-				(margins 0.9525 0.9525 0.9525 0.9525)
-				(span 1 1)
-				(fill
-					(type none)
-				)
-				(effects
-					(font
-						(size 1.27 1.27)
-					)
-					(justify left top)
-				)
-			)
-			(table_cell "0.2"
-				(exclude_from_sim no)
-				(at 105.45 50.17 0)
-				(size 27.7 4.45)
+				(at 93.98 50.17 0)
+				(size 10.9 4.45)
+				(margins 0.9525 0.9525 0.9525 0.9525)
+				(span 1 1)
+				(fill
+					(type none)
+				)
+				(effects
+					(font
+						(size 1.27 1.27)
+					)
+					(justify left top)
+				)
+			)
+			(table_cell "0.3"
+				(exclude_from_sim no)
+				(at 104.88 50.17 0)
+				(size 31.3 4.45)
 				(margins 0.9525 0.9525 0.9525 0.9525)
 				(span 1 1)
@@
 			(table_cell "PWR In"
 				(exclude_from_sim no)
-				(at 95.25 54.62 0)
-				(size 10.2 4.45)
+				(at 93.98 54.62 0)
+				(size 10.9 4.45)
 				(margins 0.9525 0.9525 0.9525 0.9525)
 				(span 1 1)
@@
 			(table_cell "+3V3"
 				(exclude_from_sim no)
-				(at 105.45 54.62 0)
-				(size 27.7 4.45)
+				(at 104.88 54.62 0)
+				(size 31.3 4.45)
 				(margins 0.9525 0.9525 0.9525 0.9525)
 				(span 1 1)
@@
 			(table_cell "I/O"
 				(exclude_from_sim no)
-				(at 95.25 59.07 0)
-				(size 10.2 4.45)
+				(at 93.98 59.07 0)
+				(size 10.9 4.45)
 				(margins 0.9525 0.9525 0.9525 0.9525)
 				(span 1 1)
@@
 			(table_cell "SCL, SDA"
 				(exclude_from_sim no)
-				(at 105.45 59.07 0)
-				(size 27.7 4.45)
+				(at 104.88 59.07 0)
+				(size 31.3 4.45)
 				(margins 0.9525 0.9525 0.9525 0.9525)
 				(span 1 1)
@@
 			(table_cell "Bus"
 				(exclude_from_sim no)
-				(at 95.25 63.52 0)
-				(size 10.2 4.45)
+				(at 93.98 63.52 0)
+				(size 10.9 4.45)
 				(margins 0.9525 0.9525 0.9525 0.9525)
 				(span 1 1)
@@
 			(table_cell "I2C Fast-mode 400kHz"
 				(exclude_from_sim no)
-				(at 105.45 63.52 0)
-				(size 27.7 4.45)
+				(at 104.88 63.52 0)
+				(size 31.3 4.45)
 				(margins 0.9525 0.9525 0.9525 0.9525)
 				(span 1 1)
@@
 			(table_cell "Pull-up"
 				(exclude_from_sim no)
-				(at 95.25 67.97 0)
-				(size 10.2 4.45)
+				(at 93.98 67.97 0)
+				(size 10.9 4.45)
 				(margins 0.9525 0.9525 0.9525 0.9525)
 				(span 1 1)
@@
 			(table_cell "1.8kΩ to +3V3"
 				(exclude_from_sim no)
-				(at 105.45 67.97 0)
-				(size 27.7 4.45)
+				(at 104.88 67.97 0)
+				(size 31.3 4.45)
 				(margins 0.9525 0.9525 0.9525 0.9525)
 				(span 1 1)
@@
 			(table_cell "Rp(min)"
 				(exclude_from_sim no)
-				(at 95.25 72.42 0)
-				(size 10.2 4.45)
+				(at 93.98 72.42 0)
+				(size 10.9 4.45)
 				(margins 0.9525 0.9525 0.9525 0.9525)
 				(span 1 1)
@@
 			(table_cell "967Ω @ 3mA IOL"
 				(exclude_from_sim no)
-				(at 105.45 72.42 0)
-				(size 27.7 4.45)
+				(at 104.88 72.42 0)
+				(size 31.3 4.45)
 				(margins 0.9525 0.9525 0.9525 0.9525)
 				(span 1 1)
@@
 			(table_cell "Source"
 				(exclude_from_sim no)
-				(at 95.25 76.87 0)
-				(size 10.2 4.45)
+				(at 93.98 76.87 0)
+				(size 10.9 4.45)
 				(margins 0.9525 0.9525 0.9525 0.9525)
 				(span 1 1)
@@
 			(table_cell "NXP UM10204 Rev 7.0 §7.1"
 				(exclude_from_sim no)
-				(at 105.45 76.87 0)
-				(size 27.7 4.45)
-				(margins 0.9525 0.9525 0.9525 0.9525)
-				(span 1 1)
+				(at 104.88 76.87 0)
+				(size 31.3 4.45)
+				(margins 0.9525 0.9525 0.9525 0.9525)
+				(span 1 1)
