File: dist/design_blocks/PartReel.kicad_blocks/stdc14.kicad_block/stdc14.kicad_sch (KiCad schematic)
At the start: 1 part, among them J1 STDC14

Commit message: 디자인 블록 재배포: g431_min 0.2(VBAT 100nF C8), emi_power_in·buck_24v_5v P13 limit_mm 실측 보정 (boardworks g431_ind24 T2)
Co-Authored-By: Claude Fable 5 <noreply@anthropic.com>
Other:
- title: STDC14 debug connector (ST-LINK V3) -> stdc14
Changed lines of the file:
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@@
 	(paper "A5")
 	(title_block
-		(title "STDC14 debug connector (ST-LINK V3)")
+		(title "stdc14")
 		(company "PartReel block")
-		(rev "0.1")
+		(rev "0.2")
 	)
 	(wire
@@
 			)
 		)
-		(column_widths 12.4 39.25)
+		(column_widths 13.3 44.5)
 		(row_heights 4.45 4.45 4.45 4.45 4.45 4.45 4.45 4.45 4.45 4.45 4.45 4.45)
 		(cells
 			(table_cell "Block"
 				(exclude_from_sim no)
-				(at 133.35 71.12 0)
-				(size 12.4 4.45)
+				(at 134.62 71.12 0)
+				(size 13.3 4.45)
 				(margins 0.9525 0.9525 0.9525 0.9525)
 				(span 1 1)
@@
 			(table_cell "STDC14 debug connector (ST-LINK V3)"
 				(exclude_from_sim no)
-				(at 145.75 71.12 0)
-				(size 39.25 4.45)
+				(at 147.92 71.12 0)
+				(size 44.5 4.45)
 				(margins 0.9525 0.9525 0.9525 0.9525)
 				(span 1 1)
@@
 			(table_cell "Rev"
 				(exclude_from_sim no)
-				(at 133.35 75.57 0)
-				(size 12.4 4.45)
-				(margins 0.9525 0.9525 0.9525 0.9525)
-				(span 1 1)
-				(fill
-					(type none)
-				)
-				(effects
-					(font
-						(size 1.27 1.27)
-					)
-					(justify left top)
-				)
-			)
-			(table_cell "0.1"
-				(exclude_from_sim no)
-				(at 145.75 75.57 0)
-				(size 39.25 4.45)
+				(at 134.62 75.57 0)
+				(size 13.3 4.45)
+				(margins 0.9525 0.9525 0.9525 0.9525)
+				(span 1 1)
+				(fill
+					(type none)
+				)
+				(effects
+					(font
+						(size 1.27 1.27)
+					)
+					(justify left top)
+				)
+			)
+			(table_cell "0.2"
+				(exclude_from_sim no)
+				(at 147.92 75.57 0)
+				(size 44.5 4.45)
 				(margins 0.9525 0.9525 0.9525 0.9525)
 				(span 1 1)
@@
 			(table_cell "PWR In"
 				(exclude_from_sim no)
-				(at 133.35 80.02 0)
-				(size 12.4 4.45)
+				(at 134.62 80.02 0)
+				(size 13.3 4.45)
 				(margins 0.9525 0.9525 0.9525 0.9525)
 				(span 1 1)
@@
 			(table_cell "+3V3, GND"
 				(exclude_from_sim no)
-				(at 145.75 80.02 0)
-				(size 39.25 4.45)
+				(at 147.92 80.02 0)
+				(size 44.5 4.45)
 				(margins 0.9525 0.9525 0.9525 0.9525)
 				(span 1 1)
@@
 			(table_cell "In"
 				(exclude_from_sim no)
-				(at 133.35 84.47 0)
-				(size 12.4 4.45)
+				(at 134.62 84.47 0)
+				(size 13.3 4.45)
 				(margins 0.9525 0.9525 0.9525 0.9525)
 				(span 1 1)
@@
 			(table_cell "SWO, UART_TX"
 				(exclude_from_sim no)
-				(at 145.75 84.47 0)
-				(size 39.25 4.45)
+				(at 147.92 84.47 0)
+				(size 44.5 4.45)
 				(margins 0.9525 0.9525 0.9525 0.9525)
 				(span 1 1)
@@
 			(table_cell "Out"
 				(exclude_from_sim no)
-				(at 133.35 88.92 0)
-				(size 12.4 4.45)
+				(at 134.62 88.92 0)
+				(size 13.3 4.45)
 				(margins 0.9525 0.9525 0.9525 0.9525)
 				(span 1 1)
@@
 			(table_cell "NRST, SWCLK, UART_RX"
 				(exclude_from_sim no)
-				(at 145.75 88.92 0)
-				(size 39.25 4.45)
+				(at 147.92 88.92 0)
+				(size 44.5 4.45)
 				(margins 0.9525 0.9525 0.9525 0.9525)
 				(span 1 1)
@@
 			(table_cell "I/O"
 				(exclude_from_sim no)
-				(at 133.35 93.37 0)
-				(size 12.4 4.45)
+				(at 134.62 93.37 0)
+				(size 13.3 4.45)
 				(margins 0.9525 0.9525 0.9525 0.9525)
 				(span 1 1)
@@
 			(table_cell "SWDIO"
 				(exclude_from_sim no)
-				(at 145.75 93.37 0)
-				(size 39.25 4.45)
+				(at 147.92 93.37 0)
+				(size 44.5 4.45)
 				(margins 0.9525 0.9525 0.9525 0.9525)
 				(span 1 1)
@@
 			(table_cell "Connector"
 				(exclude_from_sim no)
-				(at 133.35 97.82 0)
-				(size 12.4 4.45)
+				(at 134.62 97.82 0)
+				(size 13.3 4.45)
 				(margins 0.9525 0.9525 0.9525 0.9525)
 				(span 1 1)
@@
 			(table_cell "FTSH-107-01-L-DV-K-A"
 				(exclude_from_sim no)
-				(at 145.75 97.82 0)
-				(size 39.25 4.45)
+				(at 147.92 97.82 0)
+				(size 44.5 4.45)
 				(margins 0.9525 0.9525 0.9525 0.9525)
 				(span 1 1)
@@
 			(table_cell "Std"
 				(exclude_from_sim no)
-				(at 133.35 102.27 0)
-				(size 12.4 4.45)
+				(at 134.62 102.27 0)
+				(size 13.3 4.45)
 				(margins 0.9525 0.9525 0.9525 0.9525)
 				(span 1 1)
@@
 			(table_cell "STDC14 (ARM10 + VCP UART)"
 				(exclude_from_sim no)
-				(at 145.75 102.27 0)
-				(size 39.25 4.45)
+				(at 147.92 102.27 0)
+				(size 44.5 4.45)
 				(margins 0.9525 0.9525 0.9525 0.9525)
 				(span 1 1)
@@
 			(table_cell "Pin 1-2"
 				(exclude_from_sim no)
-				(at 133.35 106.72 0)
-				(size 12.4 4.45)
+				(at 134.62 106.72 0)
+				(size 13.3 4.45)
 				(margins 0.9525 0.9525 0.9525 0.9525)
 				(span 1 1)
@@
 			(table_cell "Reserved - do not connect"
 				(exclude_from_sim no)
-				(at 145.75 106.72 0)
-				(size 39.25 4.45)
+				(at 147.92 106.72 0)
+				(size 44.5 4.45)
 				(margins 0.9525 0.9525 0.9525 0.9525)
 				(span 1 1)
@@
 			(table_cell "Pin 9-10"
 				(exclude_from_sim no)
-				(at 133.35 111.17 0)
-				(size 12.4 4.45)
+				(at 134.62 111.17 0)
+				(size 13.3 4.45)
 				(margins 0.9525 0.9525 0.9525 0.9525)
 				(span 1 1)
@@
 			(table_cell "JTAG only - NC for SWD"
 				(exclude_from_sim no)
-				(at 145.75 111.17 0)
-				(size 39.25 4.45)
+				(at 147.92 111.17 0)
+				(size 44.5 4.45)
 				(margins 0.9525 0.9525 0.9525 0.9525)
 				(span 1 1)
@@
 			(table_cell "Pin 11"
 				(exclude_from_sim no)
-				(at 133.35 115.62 0)
-				(size 12.4 4.45)
+				(at 134.62 115.62 0)
+				(size 13.3 4.45)
 				(margins 0.9525 0.9525 0.9525 0.9525)
 				(span 1 1)
@@
 			(table_cell "GNDDetect - GND"
 				(exclude_from_sim no)
-				(at 145.75 115.62 0)
-				(size 39.25 4.45)
+				(at 147.92 115.62 0)
+				(size 44.5 4.45)
 				(margins 0.9525 0.9525 0.9525 0.9525)
 				(span 1 1)
@@
 			(table_cell "Source"
 				(exclude_from_sim no)
-				(at 133.35 120.07 0)
-				(size 12.4 4.45)
+				(at 134.62 120.07 0)
+				(size 13.3 4.45)
 				(margins 0.9525 0.9525 0.9525 0.9525)
 				(span 1 1)
@@
 			(table_cell "ST UM2448 Rev 9 Table 6"
 				(exclude_from_sim no)
-				(at 145.75 120.07 0)
-				(size 39.25 4.45)
-				(margins 0.9525 0.9525 0.9525 0.9525)
-				(span 1 1)
+				(at 147.92 120.07 0)
+				(size 44.5 4.45)
+				(margins 0.9525 0.9525 0.9525 0.9525)
+				(span 1 1)
