File: dist/design_blocks/PartReel.kicad_blocks/swd_uart_hdr254.kicad_block/swd_uart_hdr254.kicad_sch (KiCad schematic)
At the start: 1 part, among them J1 Header 1x8 2.54

Commit message: 디자인 블록 재배포: g431_min 0.2(VBAT 100nF C8), emi_power_in·buck_24v_5v P13 limit_mm 실측 보정 (boardworks g431_ind24 T2)
Co-Authored-By: Claude Fable 5 <noreply@anthropic.com>
Other:
- title: SWD+UART debug header (2.54mm 1x8) -> swd_uart_hdr254
Changed lines of the file:
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@@
 	(paper "A5")
 	(title_block
-		(title "SWD+UART debug header (2.54mm 1x8)")
+		(title "swd_uart_hdr254")
 		(company "PartReel block")
 		(rev "0.1")
@@
 			)
 		)
-		(column_widths 10.2 38.2)
+		(column_widths 10.9 43.3)
 		(row_heights 4.45 4.45 4.45 4.45 4.45 4.45 4.45 4.45 4.45 4.45 4.45)
 		(cells
 			(table_cell "Block"
 				(exclude_from_sim no)
-				(at 111.76 71.12 0)
-				(size 10.2 4.45)
+				(at 121.92 68.58 0)
+				(size 10.9 4.45)
 				(margins 0.9525 0.9525 0.9525 0.9525)
 				(span 1 1)
@@
 			(table_cell "SWD+UART debug header (2.54mm 1x8)"
 				(exclude_from_sim no)
-				(at 121.96 71.12 0)
-				(size 38.2 4.45)
+				(at 132.82 68.58 0)
+				(size 43.3 4.45)
 				(margins 0.9525 0.9525 0.9525 0.9525)
 				(span 1 1)
@@
 			(table_cell "Rev"
 				(exclude_from_sim no)
-				(at 111.76 75.57 0)
-				(size 10.2 4.45)
+				(at 121.92 73.03 0)
+				(size 10.9 4.45)
 				(margins 0.9525 0.9525 0.9525 0.9525)
 				(span 1 1)
@@
 			(table_cell "0.1"
 				(exclude_from_sim no)
-				(at 121.96 75.57 0)
-				(size 38.2 4.45)
+				(at 132.82 73.03 0)
+				(size 43.3 4.45)
 				(margins 0.9525 0.9525 0.9525 0.9525)
 				(span 1 1)
@@
 			(table_cell "PWR In"
 				(exclude_from_sim no)
-				(at 111.76 80.02 0)
-				(size 10.2 4.45)
+				(at 121.92 77.48 0)
+				(size 10.9 4.45)
 				(margins 0.9525 0.9525 0.9525 0.9525)
 				(span 1 1)
@@
 			(table_cell "+3V3, GND"
 				(exclude_from_sim no)
-				(at 121.96 80.02 0)
-				(size 38.2 4.45)
+				(at 132.82 77.48 0)
+				(size 43.3 4.45)
 				(margins 0.9525 0.9525 0.9525 0.9525)
 				(span 1 1)
@@
 			(table_cell "In"
 				(exclude_from_sim no)
-				(at 111.76 84.47 0)
-				(size 10.2 4.45)
+				(at 121.92 81.93 0)
+				(size 10.9 4.45)
 				(margins 0.9525 0.9525 0.9525 0.9525)
 				(span 1 1)
@@
 			(table_cell "SWO, UART_TX"
 				(exclude_from_sim no)
-				(at 121.96 84.47 0)
-				(size 38.2 4.45)
+				(at 132.82 81.93 0)
+				(size 43.3 4.45)
 				(margins 0.9525 0.9525 0.9525 0.9525)
 				(span 1 1)
@@
 			(table_cell "Out"
 				(exclude_from_sim no)
-				(at 111.76 88.92 0)
-				(size 10.2 4.45)
+				(at 121.92 86.38 0)
+				(size 10.9 4.45)
 				(margins 0.9525 0.9525 0.9525 0.9525)
 				(span 1 1)
@@
 			(table_cell "NRST, SWCLK, UART_RX"
 				(exclude_from_sim no)
-				(at 121.96 88.92 0)
-				(size 38.2 4.45)
+				(at 132.82 86.38 0)
+				(size 43.3 4.45)
 				(margins 0.9525 0.9525 0.9525 0.9525)
 				(span 1 1)
@@
 			(table_cell "I/O"
 				(exclude_from_sim no)
-				(at 111.76 93.37 0)
-				(size 10.2 4.45)
+				(at 121.92 90.83 0)
+				(size 10.9 4.45)
 				(margins 0.9525 0.9525 0.9525 0.9525)
 				(span 1 1)
@@
 			(table_cell "SWDIO"
 				(exclude_from_sim no)
-				(at 121.96 93.37 0)
-				(size 38.2 4.45)
+				(at 132.82 90.83 0)
+				(size 43.3 4.45)
 				(margins 0.9525 0.9525 0.9525 0.9525)
 				(span 1 1)
@@
 			(table_cell "Pin 1-4"
 				(exclude_from_sim no)
-				(at 111.76 97.82 0)
-				(size 10.2 4.45)
+				(at 121.92 95.28 0)
+				(size 10.9 4.45)
 				(margins 0.9525 0.9525 0.9525 0.9525)
 				(span 1 1)
@@
 			(table_cell "3V3 / SWDIO / SWCLK / NRST"
 				(exclude_from_sim no)
-				(at 121.96 97.82 0)
-				(size 38.2 4.45)
+				(at 132.82 95.28 0)
+				(size 43.3 4.45)
 				(margins 0.9525 0.9525 0.9525 0.9525)
 				(span 1 1)
@@
 			(table_cell "Pin 5-8"
 				(exclude_from_sim no)
-				(at 111.76 102.27 0)
-				(size 10.2 4.45)
+				(at 121.92 99.73 0)
+				(size 10.9 4.45)
 				(margins 0.9525 0.9525 0.9525 0.9525)
 				(span 1 1)
@@
 			(table_cell "SWO / UART_TX / UART_RX / GND"
 				(exclude_from_sim no)
-				(at 121.96 102.27 0)
-				(size 38.2 4.45)
+				(at 132.82 99.73 0)
+				(size 43.3 4.45)
 				(margins 0.9525 0.9525 0.9525 0.9525)
 				(span 1 1)
@@
 			(table_cell "Use"
 				(exclude_from_sim no)
-				(at 111.76 106.72 0)
-				(size 10.2 4.45)
+				(at 121.92 104.18 0)
+				(size 10.9 4.45)
 				(margins 0.9525 0.9525 0.9525 0.9525)
 				(span 1 1)
@@
 			(table_cell "ST-LINK V3 adapter jumpers"
 				(exclude_from_sim no)
-				(at 121.96 106.72 0)
-				(size 38.2 4.45)
+				(at 132.82 104.18 0)
+				(size 43.3 4.45)
 				(margins 0.9525 0.9525 0.9525 0.9525)
 				(span 1 1)
@@
 			(table_cell "Order"
 				(exclude_from_sim no)
-				(at 111.76 111.17 0)
-				(size 10.2 4.45)
+				(at 121.92 108.63 0)
+				(size 10.9 4.45)
 				(margins 0.9525 0.9525 0.9525 0.9525)
 				(span 1 1)
@@
 			(table_cell "PartReel convention"
 				(exclude_from_sim no)
-				(at 121.96 111.17 0)
-				(size 38.2 4.45)
+				(at 132.82 108.63 0)
+				(size 43.3 4.45)
 				(margins 0.9525 0.9525 0.9525 0.9525)
 				(span 1 1)
@@
 			(table_cell "Signals"
 				(exclude_from_sim no)
-				(at 111.76 115.62 0)
-				(size 10.2 4.45)
+				(at 121.92 113.08 0)
+				(size 10.9 4.45)
 				(margins 0.9525 0.9525 0.9525 0.9525)
 				(span 1 1)
@@
 			(table_cell "Arm UG 101636 (SWD)"
 				(exclude_from_sim no)
-				(at 121.96 115.62 0)
-				(size 38.2 4.45)
-				(margins 0.9525 0.9525 0.9525 0.9525)
-				(span 1 1)
+				(at 132.82 113.08 0)
+				(size 43.3 4.45)
+				(margins 0.9525 0.9525 0.9525 0.9525)
+				(span 1 1)
