File: dist/design_blocks/PartReel.kicad_blocks/usb_c_5v.kicad_block/usb_c_5v.kicad_sch (KiCad schematic)
At the start: 4 parts, among them J1 USB-C 16P

Commit message: 디자인 블록 재배포: g431_min 0.2(VBAT 100nF C8), emi_power_in·buck_24v_5v P13 limit_mm 실측 보정 (boardworks g431_ind24 T2)
Co-Authored-By: Claude Fable 5 <noreply@anthropic.com>
Other:
- title: USB-C 5V power input (UFP sink) -> usb_c_5v
Changed lines of the file:
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@@
 	(generator "partreel-block")
 	(generator_version "1.0")
-	(paper "A5")
+	(paper "A4")
 	(title_block
-		(title "USB-C 5V power input (UFP sink)")
+		(title "usb_c_5v")
 		(company "PartReel block")
-		(rev "0.2")
+		(rev "0.4")
 	)
 	(wire
@@
 			)
 		)
-		(column_widths 13.5 35.05)
+		(column_widths 14.5 39.7)
 		(row_heights 4.45 4.45 4.45 4.45 4.45 4.45 4.45 4.45 4.45 4.45)
 		(cells
 			(table_cell "Block"
 				(exclude_from_sim no)
-				(at 46.99 86.36 0)
-				(size 13.5 4.45)
+				(at 152.4 35.56 0)
+				(size 14.5 4.45)
 				(margins 0.9525 0.9525 0.9525 0.9525)
 				(span 1 1)
@@
 			(table_cell "USB-C 5V power input (UFP sink)"
 				(exclude_from_sim no)
-				(at 60.49 86.36 0)
-				(size 35.05 4.45)
+				(at 166.9 35.56 0)
+				(size 39.7 4.45)
 				(margins 0.9525 0.9525 0.9525 0.9525)
 				(span 1 1)
@@
 			(table_cell "Rev"
 				(exclude_from_sim no)
-				(at 46.99 90.81 0)
-				(size 13.5 4.45)
-				(margins 0.9525 0.9525 0.9525 0.9525)
-				(span 1 1)
-				(fill
-					(type none)
-				)
-				(effects
-					(font
-						(size 1.27 1.27)
-					)
-					(justify left top)
-				)
-			)
-			(table_cell "0.2"
-				(exclude_from_sim no)
-				(at 60.49 90.81 0)
-				(size 35.05 4.45)
+				(at 152.4 40.01 0)
+				(size 14.5 4.45)
+				(margins 0.9525 0.9525 0.9525 0.9525)
+				(span 1 1)
+				(fill
+					(type none)
+				)
+				(effects
+					(font
+						(size 1.27 1.27)
+					)
+					(justify left top)
+				)
+			)
+			(table_cell "0.4"
+				(exclude_from_sim no)
+				(at 166.9 40.01 0)
+				(size 39.7 4.45)
 				(margins 0.9525 0.9525 0.9525 0.9525)
 				(span 1 1)
@@
 			(table_cell "PWR Out"
 				(exclude_from_sim no)
-				(at 46.99 95.26 0)
-				(size 13.5 4.45)
+				(at 152.4 44.46 0)
+				(size 14.5 4.45)
 				(margins 0.9525 0.9525 0.9525 0.9525)
 				(span 1 1)
@@
 			(table_cell "+5V, GND"
 				(exclude_from_sim no)
-				(at 60.49 95.26 0)
-				(size 35.05 4.45)
+				(at 166.9 44.46 0)
+				(size 39.7 4.45)
 				(margins 0.9525 0.9525 0.9525 0.9525)
 				(span 1 1)
@@
 			(table_cell "I/O"
 				(exclude_from_sim no)
-				(at 46.99 99.71 0)
-				(size 13.5 4.45)
+				(at 152.4 48.91 0)
+				(size 14.5 4.45)
 				(margins 0.9525 0.9525 0.9525 0.9525)
 				(span 1 1)
@@
 			(table_cell "USB_DM, USB_DP"
 				(exclude_from_sim no)
-				(at 60.49 99.71 0)
-				(size 35.05 4.45)
+				(at 166.9 48.91 0)
+				(size 39.7 4.45)
 				(margins 0.9525 0.9525 0.9525 0.9525)
 				(span 1 1)
@@
 			(table_cell "Input"
 				(exclude_from_sim no)
-				(at 46.99 104.16 0)
-				(size 13.5 4.45)
+				(at 152.4 53.36 0)
+				(size 14.5 4.45)
 				(margins 0.9525 0.9525 0.9525 0.9525)
 				(span 1 1)
@@
 			(table_cell "USB-C VBUS 5V"
 				(exclude_from_sim no)
-				(at 60.49 104.16 0)
-				(size 35.05 4.45)
+				(at 166.9 53.36 0)
+				(size 39.7 4.45)
 				(margins 0.9525 0.9525 0.9525 0.9525)
 				(span 1 1)
@@
 			(table_cell "Role"
 				(exclude_from_sim no)
-				(at 46.99 108.61 0)
-				(size 13.5 4.45)
+				(at 152.4 57.81 0)
+				(size 14.5 4.45)
 				(margins 0.9525 0.9525 0.9525 0.9525)
 				(span 1 1)
@@
 			(table_cell "UFP sink (Rd 5.1k)"
 				(exclude_from_sim no)
-				(at 60.49 108.61 0)
-				(size 35.05 4.45)
+				(at 166.9 57.81 0)
+				(size 39.7 4.45)
 				(margins 0.9525 0.9525 0.9525 0.9525)
 				(span 1 1)
@@
 			(table_cell "Data"
 				(exclude_from_sim no)
-				(at 46.99 113.06 0)
-				(size 13.5 4.45)
+				(at 152.4 62.26 0)
+				(size 14.5 4.45)
 				(margins 0.9525 0.9525 0.9525 0.9525)
 				(span 1 1)
@@
 			(table_cell "USB 2.0 D+/D- pass-through"
 				(exclude_from_sim no)
-				(at 60.49 113.06 0)
-				(size 35.05 4.45)
+				(at 166.9 62.26 0)
+				(size 39.7 4.45)
 				(margins 0.9525 0.9525 0.9525 0.9525)
 				(span 1 1)
@@
 			(table_cell "ESD"
 				(exclude_from_sim no)
-				(at 46.99 117.51 0)
-				(size 13.5 4.45)
+				(at 152.4 66.71 0)
+				(size 14.5 4.45)
 				(margins 0.9525 0.9525 0.9525 0.9525)
 				(span 1 1)
@@
 			(table_cell "USBLC6-2P6 flow-through (CV2)"
 				(exclude_from_sim no)
-				(at 60.49 117.51 0)
-				(size 35.05 4.45)
+				(at 166.9 66.71 0)
+				(size 39.7 4.45)
 				(margins 0.9525 0.9525 0.9525 0.9525)
 				(span 1 1)
@@
 			(table_cell "TODO rev B"
 				(exclude_from_sim no)
-				(at 46.99 121.96 0)
-				(size 13.5 4.45)
+				(at 152.4 71.16 0)
+				(size 14.5 4.45)
 				(margins 0.9525 0.9525 0.9525 0.9525)
 				(span 1 1)
@@
 			(table_cell "ESD array + polyfuse"
 				(exclude_from_sim no)
-				(at 60.49 121.96 0)
-				(size 35.05 4.45)
+				(at 166.9 71.16 0)
+				(size 39.7 4.45)
 				(margins 0.9525 0.9525 0.9525 0.9525)
 				(span 1 1)
@@
 			(table_cell "Source"
 				(exclude_from_sim no)
-				(at 46.99 126.41 0)
-				(size 13.5 4.45)
+				(at 152.4 75.61 0)
+				(size 14.5 4.45)
 				(margins 0.9525 0.9525 0.9525 0.9525)
 				(span 1 1)
@@
 			(table_cell "USB Type-C spec R2.2 4.5.1.2.3"
 				(exclude_from_sim no)
-				(at 60.49 126.41 0)
-				(size 35.05 4.45)
-				(margins 0.9525 0.9525 0.9525 0.9525)
-				(span 1 1)
+				(at 166.9 75.61 0)
+				(size 39.7 4.45)
+				(margins 0.9525 0.9525 0.9525 0.9525)
+				(span 1 1)
